File: fuente-lineal.kicad_sch (KiCad schematic)
At the start: 38 parts, among them J1 Conn_01x03, J2 Conn_01x03, J3 Conn_01x01, J4 Conn_01x01, J5 Conn_01x01, J6 Conn_01x01, J7 Conn_01x01, J8 Conn_01x01, J9 Conn_01x02, U1 LM7805_TO220

Commit message: completando version v1.1.0
Parts:
- removed C10, C9: 2200uF, Capacitor_THT:CP_Radial_D13.0mm_P5.00mm, symbol Device:C_Polarized_US
- removed C3, C4: 2200uF, Capacitor_THT:CP_Radial_D16.0mm_P7.50mm, symbol Device:C_Polarized_US
- removed J3, J4, J5, J6, J7, J8: Conn_01x01, Connector_Pin:Pin_D1.1mm_L8.5mm_W2.5mm_FlatFork, symbol Connector_Generic:Conn_01x01
- added C13, C14, C3, C4: 100nF, Capacitor_THT:C_Disc_D5.0mm_W2.5mm_P5.00mm, symbol Device:C
- added J3: Conn_01x03, TerminalBlock_MetzConnect:TerminalBlock_MetzConnect_Type073_RT02603HBLU_1x03_P5.08mm_Horizontal, symbol Connector_Generic:Conn_01x03
- added J6: Conn_01x03, Connector_PinHeader_2.54mm:PinHeader_1x03_P2.54mm_Vertical, symbol Connector_Generic:Conn_01x03
- added R1: 34, symbol Device:R_US
- added R2: 30, symbol Device:R_US
- C1, C2, C5, C6: footprint Capacitor_THT:CP_Radial_D16.0mm_P7.50mm -> Capacitor_THT:CP_Radial_D13.0mm_P5.00mm; LCSC Part (none) -> C43275; Manufacturer (none) -> CX(Dongguan Chengxing Elec); Mfr. Part (none) -> GR228M035J25RR0VH4FP0; Price (none) -> 0.19; V 63V -> 35V
- C11: value 0.33uF -> 2.2uF; footprint Capacitor_THT:CP_Radial_D6.3mm_P2.50mm -> Capacitor_THT:CP_Radial_D5.0mm_P2.00mm; LCSC Part (none) -> C442804; Manufacturer (none) -> Ymin; Mfr. Part (none) -> LKMB0901E2R2MF; Price (none) -> 0.0334
- C12: footprint Capacitor_THT:C_Disc_D6.0mm_W2.5mm_P5.00mm -> Capacitor_THT:C_Disc_D5.0mm_W2.5mm_P5.00mm; LCSC Part (none) -> C254094; Manufacturer (none) -> Dersonic; Mfr. Part (none) -> CC1H104ZC74D3F5O30MN; Price (none) -> 0.0158
- C7: footprint Capacitor_THT:CP_Radial_D13.0mm_P5.00mm -> Capacitor_THT:CP_Radial_D12.5mm_P5.00mm; LCSC Part (none) -> C134573; Manufacturer (none) -> Lelon; Mfr. Part (none) -> RGA222M1EBK-1325; Price (none) -> 0.21
- C8: LCSC Part (none) -> C43275; Manufacturer (none) -> CX(Dongguan Chengxing Elec); Mfr. Part (none) -> GR228M035J25RR0VH4FP0; Price (none) -> 0.19
- D1, D2, D3, D4: value 6A10 -> 1N5404; footprint Diode_THT:D_P600_R-6_P20.00mm_Horizontal -> Diode_THT:D_DO-27_P15.24mm_Horizontal; LCSC Part (none) -> C5365389; Manufacturer (none) -> JUXING; Mfr. Part (none) -> 1N5404; Price (none) -> 0.0470
- D5, D6, D7, D8: LCSC Part (none) -> C5365389; Manufacturer (none) -> JUXING; Mfr. Part (none) -> 1N5404; Price (none) -> 0.0470
- H1, H2, H3, H4: now left out of the parts list
- U1: LCSC Part (none) -> C427632; Manufacturer (none) -> UTC(Unisonic Tech); Mfr. Part (none) -> LM7805AL-TA3-T; Price (none) -> 0.1707
- V10, V6, V7, V8: now not fitted
Connections:
- net GND: now also C13.2, C14.1, C3.2, C4.1, J3.2 (Pin_2), J6.2 (Pin_2), R1.2, R2.1
- net V1i: now also D1.2 (A), D2.1 (K); no longer D3.1 (K), D4.2 (A)
- net V2i: now also D3.2 (A), D4.1 (K); no longer D1.1 (K), D2.2 (A)
- net Vo2n: now also C4.2, J6.3 (Pin_3)
- net Vo2p: now also C3.1, J6.1 (Pin_1)
- net Von: now also D2.2 (A), D4.2 (A), C14.2, J3.3 (Pin_3), R2.2; no longer D1.2 (A), D3.2 (A)
- net Vop: now also D1.1 (K), D3.1 (K), C13.1, J3.1 (Pin_1), R1.1; no longer D2.1 (K), D4.1 (K)
Other:
- note added: "Los componentes marcados con X son usados solo para simulacion"
- moved on the sheet: C8, J9
